File: main.brd (EAGLE design)
At the start: 62 x 30 mm, 47 parts, among them IC1 HDC1000, IC2 TPS2115, IC3 BQ24080-Q1,, K1 TS-1109

Commit message: End PCB Routing
Parts:
- removed C16, C17: (no value), My_RLC:C0603
- removed JP1: (no value), pinhead:1X02
- removed K1: TS-1109, Seeed-OPL-Button:SW4-6.0X6.0X5.0MM
- added IC4: SI1147, silabs:QFN-10
- added JP3: (no value), pinhead:1X04
- added JP4: (no value), pinhead:1X03
- added LED1: (no value), led:LED3MM
- added R13, R14, R15: (no value), My_RLC:R0603
- moved C18 52.6 mm to (45.4, 5.00), turned to 270 degrees
- moved C19 4.03 mm to (54.2, 26.9), turned to 270 degrees
- moved C8 2.78 mm to (6.00, 26.3), turned to 90 degrees
- moved C1 2.61 mm to (1.41, 20.0)
Connections:
- removed net USR_B: K1.1
- new net N$16: LED1.A, R13.1
- new net N$17: IC4.9, LED1.K
- new net N$20: JP4.2, R14.2
- new net RX: JP3.3, U$1.15
- new net SI_INT: IC4.4
- new net TX: JP3.2, U$1.16
- net +3V3: now also IC4.3, JP3.1, R13.2; no longer C16.1, C17.1
- net CE: now also R14.1, R15.1; no longer U$1.4
- net GND: now also IC4.8, JP3.4, JP4.3, R15.2; no longer C16.2, C17.2, JP1.2, K1.2, K1.3
- net SCL: now also IC4.2
- net SDA: now also IC4.1
- net VDD: now also JP4.1; no longer JP1.1
Routing:
- net TX: track 0.00 -> 43.7 mm, vias 0 -> 1
- net RX: track 0.00 -> 42.7 mm, vias 0 -> 1
- net N$20: track 0.00 -> 29.4 mm, vias 0 -> 1
- net WAKEUP_B: track 0.00 -> 29.4 mm, vias 0 -> 1
- net +3V3: track 142.3 -> 167.1 mm, vias 9 -> 10
- net SCL: track 64.2 -> 76.6 mm, vias 1 -> 3
- net SDA: track 62.5 -> 72.0 mm, vias 2 -> 4
- net N$16: track 0.00 -> 8.79 mm
- net N$17: track 0.00 -> 6.90 mm
- net CE: track 18.1 -> 14.9 mm
- net VDD: track 31.3 -> 33.9 mm
- net ST1: track 21.9 -> 23.8 mm
- net ST2: track 21.3 -> 23.1 mm
- net GND: vias 21 -> 109
Other:
- outline, holes or cut-outs redrawn
- board text added: "3.3V"
- board text added: "GND"
- board text added: "RX"
- board text added: "TX"
