File: main.sch (EAGLE design)
At the start: 47 parts, among them IC1 HDC1000, IC2 TPS2115, IC3 BQ24080-Q1,, K1 TS-1109

Commit message: End PCB Routing
Parts:
- removed C16, C17: (no value), My_RLC:CAP0603
- removed JP1: (no value), pinhead:PINHD-1X2
- removed K1: TS-1109, Seeed-OPL-Button:DIP-BUTTON-4P
- added IC4: SI1147, silabs:SI1147
- added JP3: (no value), pinhead:PINHD-1X4
- added JP4: (no value), pinhead:PINHD-1X3
- added LED1: (no value), led:LED3MM
- added R13, R14, R15: (no value), My_RLC:RES0603
Connections:
- removed net USR_B: K1.A0
- new net N$16: LED1.A, R13.P$1
- new net N$17: IC4.LED1, LED1.C
- new net N$20: JP4.2, R14.P$2
- new net RX: JP3.3, U$1.15
- new net SI_INT: IC4.INT
- new net TX: JP3.2, U$1.16
- net +3V3: now also IC4.VDD, JP3.1, R13.P$2; no longer C16.P$1, C17.P$1
- net CE: now also R14.P$1, R15.P$1; no longer U$1.4
- net GND: now also IC4.GND, JP3.4, JP4.3, R15.P$2; no longer C16.P$2, C17.P$2, JP1.2, K1.B0, K1.B1
- net SCL: now also IC4.SCL
- net SDA: now also IC4.SDA
- net VDD: now also JP4.1; no longer JP1.1
